File: hotshot_keyboard.kicad_pcb (KiCad board)
At the start: 2 copper layers, 86.5 x 38.1 mm, 25 parts, among them SW1 SW_Push, U1 ATmega32U4-AU, Y1 Crystal_GND24_Small

Commit message: update pcb
Parts:
- removed C1, C2: 22pF, Capacitor_SMD:C_0805_2012Metric
- removed C3: 1uF, Capacitor_SMD:C_0805_2012Metric
- removed C4, C5, C6, C7: 0.1uF, Capacitor_SMD:C_0805_2012Metric
- removed C8: 10uF, Capacitor_SMD:C_0805_2012Metric
- removed D1, D2, D3, D4: D_Small, Diode_SMD:D_SOD-123
- removed F1: 500mA, Fuse:Fuse_1206_3216Metric
- removed MX2, MX3, MX4: MX-NoLED, MX_Alps_Hybrid:MX-1U
- removed USB1: Molex-0548190589, random-keyboard-parts:Molex-0548190589
- added MX40: ', MX_Alps_Hybrid:MX-1U-NoLED, F.Cu at (247.7, 61.9)
- added MX41: ENTER, MX_Alps_Hybrid:MX-2.25U-NoLED, F.Cu at (278.6, 61.9)
- added MX42: LSHIFT, MX_Alps_Hybrid:MX-2.25U-NoLED, F.Cu at (35.7, 81.0)
- added MX43: Z, MX_Alps_Hybrid:MX-1U-NoLED, F.Cu at (66.7, 81.0)
- added MX44: X, MX_Alps_Hybrid:MX-1U-NoLED, F.Cu at (85.7, 81.0)
- added MX45: C, MX_Alps_Hybrid:MX-1U-NoLED, F.Cu at (104.8, 81.0)
- added MX46: V, MX_Alps_Hybrid:MX-1U-NoLED, F.Cu at (123.8, 81.0)
- added MX47: B, MX_Alps_Hybrid:MX-1U-NoLED, F.Cu at (142.9, 81.0)
- added MX48: N, MX_Alps_Hybrid:MX-1U-NoLED, F.Cu at (161.9, 81.0)
- added MX49: M, MX_Alps_Hybrid:MX-1U-NoLED, F.Cu at (181.0, 81.0)
- added MX50: ,<, MX_Alps_Hybrid:MX-1U-NoLED, F.Cu at (200.0, 81.0)
- added MX51: .>, MX_Alps_Hybrid:MX-1U-NoLED, F.Cu at (219.1, 81.0)
- added MX52: /?, MX_Alps_Hybrid:MX-1U-NoLED, F.Cu at (238.1, 81.0)
- added MX53: RSHIFT, MX_Alps_Hybrid:MX-2.75U-NoLED, F.Cu at (273.8, 81.0)
- added MX54: LCTRL, MX_Alps_Hybrid:MX-1.25U-NoLED, F.Cu at (26.2, 100.0)
- added MX55: LCMD, MX_Alps_Hybrid:MX-1.25U-NoLED, F.Cu at (50.0, 100.0)
- added MX56: LALT, MX_Alps_Hybrid:MX-1.25U-NoLED, F.Cu at (73.8, 100.0)
- added MX57: SPACE, MX_Alps_Hybrid:MX-6.25U-NoLED, F.Cu at (145.3, 100.0)
- added MX58: RALT, MX_Alps_Hybrid:MX-1.25U-NoLED, F.Cu at (216.7, 100.0)
- added MX59: RCMD, MX_Alps_Hybrid:MX-1.25U-NoLED, F.Cu at (240.5, 100.0)
- added MX60: FN, MX_Alps_Hybrid:MX-1.25U-NoLED, F.Cu at (264.3, 100.0)
- added MX61: RCTRL, MX_Alps_Hybrid:MX-1.25U-NoLED, F.Cu at (288.1, 100.0)
- added R5: 5.1K, Resistor_SMD:R_0805_2012Metric_Pad1.20x1.40mm_HandSolder, B.Cu at (239.5, 21.4)
- added R6: 5.1k, Resistor_SMD:R_0805_2012Metric_Pad1.20x1.40mm_HandSolder, B.Cu at (245.1, 20.6)
- added U2: PRTR5V0U2X, random-keyboard-parts:SOT143B, B.Cu at (243.7, 25.4)
- MX1: value MX-NoLED -> ESC; footprint MX_Alps_Hybrid:MX-1U -> MX_Alps_Hybrid:MX-1U-NoLED
- R1, R3: footprint Resistor_SMD:R_0805_2012Metric -> Resistor_SMD:R_0805_2012Metric_Pad1.20x1.40mm_HandSolder; moved to B.Cu
- R2: value 22 -> 10k; footprint Resistor_SMD:R_0805_2012Metric -> Resistor_SMD:R_0805_2012Metric_Pad1.20x1.40mm_HandSolder; moved to B.Cu
- R4: value 10k -> 22; footprint Resistor_SMD:R_0805_2012Metric -> Resistor_SMD:R_0805_2012Metric_Pad1.20x1.40mm_HandSolder; moved to B.Cu
- SW1: footprint random-keyboard-parts:SKQG-1155865 -> Button_Switch_SMD:SW_SPST_SKQG_WithStem; moved to B.Cu
- Y1: value Crystal_GND24_Small -> XTAL; footprint Crystal:Crystal_SMD_3225-4Pin_3.2x2.5mm -> Crystal:Crystal_SMD_3225-4Pin_3.2x2.5mm_HandSoldering
- moved MX1 161.5 mm to (23.8, 23.8)
- moved Y1 111.9 mm to (172.9, 145.7)
- moved R3 104.4 mm to (177.8, 133.6), turned to 0 degrees
- moved R2 97.3 mm to (181.6, 127.0), turned to 0 degrees
- moved U1 94.5 mm to (144.5, 138.1)
- moved R4 85.8 mm to (177.8, 130.7)
- moved R1 84.7 mm to (159.5, 129.4)
- moved SW1 69.2 mm to (149.3, 123.3)
Connections:
- net Net-(C1-Pad1) renamed /XTAL1
- net Net-(C2-Pad1) renamed /XTAL2
- net Net-(R1-Pad1) renamed /RESET
- net Net-(U1-Pad10) renamed /MOSI
- net Net-(U1-Pad11) renamed /MISO
- net Net-(U1-Pad37) renamed /ROW4
- net Net-(U1-Pad38) renamed /ROW3
- net Net-(U1-Pad39) renamed /ROW2
- net Net-(U1-Pad40) renamed /ROW1
- net Net-(U1-Pad41) renamed /ROW0
- net Net-(U1-Pad9) renamed /SCK
- MX1 pad 1: COL0 -> /COL0
- R2 pad 2: D+ -> GND
- R3 pad 1: D- -> /D-
- R3 pad 2: Net-(R3-Pad2) -> Net-(J2-PadA7)
- R4 pad 1: GND -> /D+
- R4 pad 2: Net-(R4-Pad2) -> Net-(J2-PadA6)
- U1 pad 12: Net-(U1-Pad12) -> /COL3
- U1 pad 15: Net-(U1-Pad15) -> GND
- U1 pad 18: Net-(U1-Pad18) -> /COL6
- U1 pad 19: Net-(U1-Pad19) -> /COL7
- U1 pad 20: Net-(U1-Pad20) -> /COL8
- U1 pad 21: Net-(U1-Pad21) -> /COL9
- U1 pad 22: Net-(U1-Pad22) -> /COL11
- U1 pad 23: Net-(U1-Pad15) -> GND
- U1 pad 24: Net-(U1-Pad24) -> +5V
- U1 pad 25: Net-(U1-Pad25) -> /COL10
- U1 pad 26: Net-(U1-Pad26) -> /COL12
- U1 pad 27: ROW0 -> /COL13
- U1 pad 28: COL1 -> /COL0
- U1 pad 29: COL0 -> /COL1
- U1 pad 3: Net-(R3-Pad2) -> /D-
- U1 pad 30: ROW1 -> /COL2
- U1 pad 31: Net-(U1-Pad31) -> /COL4
- U1 pad 32: Net-(U1-Pad32) -> /COL5
- U1 pad 33: Net-(R4-Pad2) -> Net-(R2-Pad1)
- U1 pad 35: Net-(U1-Pad15) -> GND
- U1 pad 4: Net-(R2-Pad1) -> /D+
- U1 pad 43: Net-(U1-Pad15) -> GND
- U1 pad 44: Net-(U1-Pad24) -> +5V
Routing:
- net D-: track 7.60 -> 0.00 mm
Other:
- board outline removed

Commit message: update pcb
Parts:
- moved U1 54.5 mm to (177.0, 94.5), turned to 180 degrees
- moved R3 45.6 mm to (186.5, 88.9)
- moved Y1 40.4 mm to (177.3, 105.6)
- moved R2 39.6 mm to (168.3, 89.7), turned to 90 degrees
- moved R4 39.6 mm to (186.5, 92.1)
- moved R1 36.4 mm to (166.7, 93.7)
- moved SW1 31.4 mm to (159.5, 93.7), turned to 180 degrees
Other:
- board outline added: 285.8 x 99.2 mm

Commit message: update pcb
Parts:
- added C5: 0.1u, Capacitor_SMD:C_0805_2012Metric_Pad1.18x1.45mm_HandSolder, B.Cu at (182.8, 103.2)
- added MX13: =+, MX_Alps_Hybrid:MX-1U-NoLED, F.Cu at (252.4, 23.8)
- added MX8: #7, MX_Alps_Hybrid:MX-1U-NoLED, F.Cu at (157.2, 23.8)
- MX57: footprint MX_Alps_Hybrid:MX-6.25U-NoLED -> MX_Alps_Hybrid:MX-6.25U-ReversedStabilizers-NoLED
- moved R4 6.05 mm to (191.5, 88.6), turned to 90 degrees
- moved R3 2.96 mm to (189.5, 88.6), turned to 90 degrees
- moved Y1 2.38 mm to (174.9, 105.6)
- moved U2 1.02 mm to (242.9, 26.0), turned to 180 degrees
- moved R6 0.89 mm to (245.5, 19.8), turned to 270 degrees
Connections:
- net Net-(J2-PadA6) renamed /DD+
- net Net-(J2-PadA7) renamed /DD-
- MX57 pad 1: /COL6 -> /COL5
- MX58 pad 1: /COL10 -> /COL9
- MX59 pad 1: /COL11 -> /COL10
- MX60 pad 1: /COL12 -> /COL11
Routing:
- net /ROW2: track 0.00 -> 238.0 mm
- net /ROW1: track 0.00 -> 228.7 mm
- net /ROW0: track 0.00 -> 228.5 mm
- net /ROW3: track 0.00 -> 208.2 mm
- net /ROW4: track 0.00 -> 195.6 mm
- net /DD-: track 0.00 -> 101.0 mm
- net /DD+: track 0.00 -> 100.8 mm
- net /COL1: track 0.00 -> 88.7 mm
- net /COL11: track 0.00 -> 86.3 mm
- net /COL2: track 0.00 -> 86.2 mm
- net /COL13: track 0.00 -> 83.4 mm
- net /COL5: track 0.00 -> 83.4 mm
- net /COL10: track 0.00 -> 83.4 mm
- net /COL0: track 0.00 -> 82.3 mm
- net /COL9: track 0.00 -> 82.3 mm
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- added copper zone on B.Cu, net GND

Commit message: update pcb zones
Parts:
- added MX26: [{, MX_Alps_Hybrid:MX-1U-NoLED, F.Cu at (242.9, 42.9)
Routing:
- net /DD-: track 101.0 -> 100.2 mm
- net /DD+: track 100.8 -> 100.2 mm
- net GND: vias 0 -> 2
- added copper zone on F.Cu, net GND

Commit message: update pcb
Parts:
- added MX27: ]}, MX_Alps_Hybrid:MX-1U-NoLED, F.Cu at (261.9, 42.9)
- added MX38: L, MX_Alps_Hybrid:MX-1U-NoLED, F.Cu at (209.6, 61.9)
- added MX39: ;:, MX_Alps_Hybrid:MX-1U-NoLED, F.Cu at (228.6, 61.9)
- moved R6 1.00 mm to (245.5, 20.8)
Routing:
- net +5V: track 6.24 -> 170.4 mm, vias 0 -> 5
- net GND: track 23.4 -> 71.3 mm
- net VCC: track 0.00 -> 28.7 mm, vias 0 -> 2
- net Net-(J2-PadA5): track 0.00 -> 5.51 mm
- net Net-(J2-PadB5): track 0.00 -> 3.45 mm

Commit message: reconfig schematics row/cols
Parts:
- moved SW1 38.9 mm to (171.1, 130.8)
- moved R1 31.4 mm to (170.6, 124.8)
Connections:
- U1 pad 1: Net-(U1-Pad1) -> /ROW3
- U1 pad 12: /COL3 -> /COL9
- U1 pad 18: /COL6 -> /COL11
- U1 pad 19: /COL7 -> /COL13
- U1 pad 20: /COL8 -> Net-(U1-Pad20)
- U1 pad 21: /COL9 -> Net-(U1-Pad21)
- U1 pad 22: /COL11 -> Net-(U1-Pad22)
- U1 pad 25: /COL10 -> /ROW4
- U1 pad 26: /COL12 -> /COL5
- U1 pad 27: /COL13 -> /COL0
- U1 pad 28: /COL0 -> /COL1
- U1 pad 29: /COL1 -> /COL2
- U1 pad 30: /COL2 -> /COL3
- U1 pad 32: /COL5 -> /COL6
- U1 pad 36: Net-(U1-Pad36) -> /ROW1
- U1 pad 37: /ROW4 -> /ROW2
- U1 pad 38: /ROW3 -> /ROW0
- U1 pad 39: /ROW2 -> /COL7
- U1 pad 40: /ROW1 -> /COL8
- U1 pad 41: /ROW0 -> /COL12
- U1 pad 8: Net-(U1-Pad8) -> /COL10
Routing:
- net GND: track 71.3 -> 211.7 mm
- net +5V: track 170.4 -> 175.2 mm
- net Net-(R2-Pad1): track 0.00 -> 3.13 mm
- removed copper zone on B.Cu, net GND
- removed copper zone on F.Cu, net GND

Commit message: update pcb route
Parts:
- moved SW1 27.7 mm to (160.0, 105.4)
- moved R1 19.9 mm to (166.4, 105.4), turned to 90 degrees
Connections:
- U1 pad 40: /COL8 -> /COL12
- U1 pad 41: /COL12 -> /COL8
Routing:
- net /COL0: track 82.3 -> 233.6 mm, vias 0 -> 1
- net /COL1: track 88.7 -> 219.1 mm, vias 0 -> 1
- net /COL13: track 83.4 -> 204.2 mm, vias 0 -> 1
- net /COL12: track 22.1 -> 137.4 mm, vias 0 -> 2
- net /ROW0: track 228.5 -> 334.1 mm, vias 0 -> 7
- net /COL2: track 86.2 -> 180.8 mm, vias 0 -> 1
- net /COL11: track 86.3 -> 179.6 mm, vias 0 -> 1
- net /ROW4: track 195.6 -> 288.1 mm
- net /ROW1: track 228.7 -> 319.3 mm, vias 0 -> 7
- net /COL3: track 64.3 -> 142.2 mm, vias 0 -> 1
- net /RESET: track 0.00 -> 76.1 mm, vias 0 -> 5
- net /COL10: track 83.4 -> 143.4 mm, vias 0 -> 1
- net /COL4: track 64.3 -> 123.2 mm, vias 0 -> 1
- net /ROW3: track 208.2 -> 263.8 mm, vias 0 -> 5
- net GND: track 211.7 -> 260.9 mm
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
Commit message: remastered pcb
Parts:
- added D12: D_Small, Diode_SMD:D_SOD-123, B.Cu at (238.9, 27.8)
- added F1: 500mA, Fuse:Fuse_1206_3216Metric_Pad1.42x1.75mm_HandSolder, B.Cu at (234.9, 33.0)
- added MX16: Q, MX_Alps_Hybrid:MX-1U-NoLED, F.Cu at (52.4, 42.9)
- added MX30: A, MX_Alps_Hybrid:MX-1U-NoLED, F.Cu at (57.1, 61.9)
- added MX4: #3, MX_Alps_Hybrid:MX-1U-NoLED, F.Cu at (81.0, 23.8)
- added MX6: #5, MX_Alps_Hybrid:MX-1U-NoLED, F.Cu at (119.1, 23.8)
- added MX7: #6, MX_Alps_Hybrid:MX-1U-NoLED, F.Cu at (138.1, 23.8)
- moved C5 4.47 mm to (186.7, 105.4), turned to 270 degrees
- moved Y1 2.86 mm to (177.8, 105.4)
- moved U1 1.12 mm to (177.8, 95.2)
- moved R2 0.79 mm to (168.9, 90.2)
- moved U2 0.71 mm to (242.6, 25.4)
- moved R6 0.66 mm to (245.1, 20.3)
- moved R5 0.55 mm to (240.0, 21.6)
- moved R3 0.36 mm to (189.2, 88.9)
- moved R4 0.36 mm to (191.8, 88.9)
Routing:
- net GND: track 260.9 -> 35.1 mm, vias 2 -> 0
- net +5V: track 208.5 -> 0.00 mm, vias 5 -> 0
- net /COL0: track 233.6 -> 82.3 mm, vias 1 -> 0
- net /COL1: track 219.1 -> 88.7 mm, vias 1 -> 0
- net /COL13: track 204.2 -> 83.4 mm, vias 1 -> 0
- net /COL12: track 137.4 -> 22.1 mm, vias 2 -> 0
- net /ROW1: track 319.3 -> 208.7 mm, vias 7 -> 0
- net /COL2: track 180.8 -> 86.2 mm, vias 1 -> 0
- net /COL11: track 179.6 -> 86.3 mm, vias 1 -> 0
- net /ROW4: track 288.1 -> 196.1 mm
- net /ROW0: track 334.1 -> 248.9 mm, vias 7 -> 0
- net /COL3: track 142.2 -> 64.3 mm, vias 1 -> 0
- net /ROW3: track 263.8 -> 189.2 mm, vias 5 -> 0
- net /RESET: track 76.1 -> 6.20 mm, vias 5 -> 0
- net /ROW2: track 282.7 -> 218.6 mm, vias 4 -> 0
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