File: hotshot_keyboard.kicad_pcb (KiCad board)
At the start: 2 copper layers, 285.8 x 99.2 mm, 47 parts, among them SW1 SW_Push, U1 ATmega32U4-AU, U2 PRTR5V0U2X, Y1 XTAL

Commit message: update pcb
Parts:
- moved SW1 49.5 mm to (209.6, 105.4)
- moved R1 36.8 mm to (203.2, 105.4), turned to 270 degrees
Routing:
- net GND: track 35.1 -> 260.6 mm, vias 0 -> 7
- net +5V: track 0.00 -> 184.6 mm, vias 0 -> 6
- net /RESET: track 6.20 -> 34.7 mm
- net /ROW3: track 189.2 -> 215.1 mm
- net /ROW1: track 208.7 -> 233.5 mm
- net /ROW2: track 218.6 -> 243.2 mm
- net VCC: track 8.50 -> 27.9 mm
- net /ROW0: track 248.9 -> 233.6 mm
- net /COL11: track 86.3 -> 97.5 mm
- net /COL13: track 83.4 -> 94.4 mm
- net /XTAL2: track 0.00 -> 10.9 mm
- net /COL9: track 82.3 -> 91.5 mm
- net /COL10: track 83.4 -> 92.5 mm
- net /SCK: track 0.00 -> 8.93 mm
- net /MOSI: track 0.00 -> 8.69 mm
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
Commit message: update left part
Parts:
- added MX36: J, MX_Alps_Hybrid:MX-1U-NoLED, F.Cu at (171.4, 61.9)
Routing:
- net /COL0: track 82.3 -> 244.7 mm, vias 0 -> 1
- net /COL1: track 88.7 -> 227.9 mm, vias 0 -> 1
- net /COL2: track 86.2 -> 201.0 mm, vias 0 -> 1
- net /COL3: track 64.3 -> 157.9 mm, vias 0 -> 1
- net /COL4: track 64.3 -> 140.2 mm, vias 0 -> 1
- net /ROW0: track 233.6 -> 298.5 mm, vias 0 -> 2
- net /ROW1: track 233.5 -> 279.3 mm, vias 0 -> 2
- net /COL5: track 83.4 -> 120.4 mm
- net /ROW4: track 196.1 -> 221.2 mm
- net /COL6: track 64.3 -> 86.0 mm, vias 0 -> 1
- net /ROW2: track 243.2 -> 260.9 mm
- net GND: track 260.6 -> 273.0 mm
- net /COL7: track 68.7 -> 75.7 mm
- net +5V: track 184.6 -> 183.9 mm

Commit message: pcb full connected
Routing:
- net /COL13: track 94.4 -> 215.2 mm, vias 0 -> 1
- net /COL12: track 26.7 -> 141.2 mm, vias 0 -> 3
- net /COL11: track 97.5 -> 189.6 mm, vias 0 -> 1
- net /ROW4: track 221.2 -> 286.9 mm
- net /COL10: track 92.5 -> 143.7 mm, vias 0 -> 1
- net /ROW3: track 215.1 -> 259.7 mm, vias 0 -> 2
- net /ROW1: track 279.3 -> 322.1 mm, vias 2 -> 6
- net /ROW0: track 298.5 -> 340.3 mm, vias 2 -> 6
- net /COL9: track 91.5 -> 115.9 mm
- net /MOSI: track 8.69 -> 31.3 mm
- net +5V: track 183.9 -> 205.8 mm
- net /ROW2: track 260.9 -> 281.9 mm, vias 0 -> 4
- net /COL8: track 69.0 -> 89.1 mm, vias 0 -> 1
- net /SCK: track 8.93 -> 28.8 mm
- net /RESET: track 34.7 -> 54.5 mm, vias 0 -> 2
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
Commit message: update diode
Parts:
- D12: value D_Small -> 1N4148
