File: SCHEMATICS & PCB/hotshot_keyboard.kicad_pcb (KiCad board)
At the start: 2 copper layers, 285.8 x 99.2 mm, 48 parts, among them SW1 SW_Push, U1 ATmega32U4-AU, U2 PRTR5V0U2X, Y1 XTAL

Commit message: add copper GND to mc crystal
Routing:
- net /COL13: track 215.2 -> 203.8 mm
- net /COL11: track 189.6 -> 179.5 mm
- net GND: track 287.9 -> 288.1 mm, vias 8 -> 10
- added copper zone on B.Cu, net GND
- added copper zone on F.Cu, net GND
